File: Projects/ESP Projects/IoT Control Board/HomeAutomation.sch (EAGLE design)
At the start: 37 parts, among them IC1 7805T, J1 OUT 1, J2 OUT 3, J3 OUT 4, J4 OUT 2, J5 POWER_JACK, K1 RELAY-SPDT-JZC-11F, K2 RELAY-SPDT-JZC-11F, K3 RELAY-SPDT-JZC-11F, K4 RELAY-SPDT-JZC-11F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

Commit message: Add files via upload
Parts:
- removed D1: 1N4004, diode:1N4004
- removed R10, R8, R9: 0.3, SparkFun-Resistors:0.3OHM-0805-1/8W-1%
- added D9: B340A-E3/61T, diode:DIODE-DO214AC
- added L1: 33µH/±20%/1.4A, SparkFun-Coils:INDUCTOR-SRN6045-33UH
- C1: value 0.33uF -> 680uf; device SparkFun-Capacitors:10UF-POLAR-RADIAL-2.5MM-KIT-25V-20% -> rcl:CPOL-EU153CLV-0405
- C2: value 0.1uF -> 220uF; device SparkFun-Capacitors:10UF-POLAR-RADIAL-2.5MM-KIT-25V-20% -> rcl:CPOL-EU153CLV-0405
- D10: value RGB -> 1N4007; device SparkFun-LED:LED-RGBPLCC-6 -> diode:DIODE-DO214AC
- D2, D3, D4: value 1N4004 -> 1N4007; device diode:1N4004 -> diode:DIODE-DO214AC
- D5, D6, D7, D8: device SparkFun-LED:LED5MM -> led:LEDCHIPLED_1206
- IC1: value 7805T -> LM2596S; device linear:7805T -> national-semiconductor:LM2596S
- J5: value POWER_JACK -> 694106301002; device SparkFun-Connectors:POWER_JACK -> DC Power Jacks:694106301002
- K1, K2, K3, K4: value RELAY-SPDT-JZC-11F -> SIEMENS_V23082; device SparkFun-Electromechanical:RELAY-SPDT-JZC-11F -> LezzetliRobotTarifleri:SIEMENS_V23082_RELAY
- R2, R3: device SparkFun-Resistors:1KOHM-HORIZ-1/4W-5% -> Resistor:R_CHIP-0402(1005-METRIC)
- R4, R5, R6, R7: device SparkFun-Resistors:1KOHM-HORIZ-1/4W-5% -> rcl:R-EU_R0805
- T1, T2, T3, T4: device transistor:2N2222 -> transistor:MMBT2222ALT1-NPN-SOT23-BEC
Connections:
- removed net D0: ESP8266.D0, R2.2, U1.DATA
- removed net D3: D8.A, ESP8266.D3, T3.B
- removed net D4: D7.A, ESP8266.D4, T4.B
- removed net N$22: D10.RED-A, R10.2
- removed net N$24: D10.GRN-A, R9.2
- removed net N$8: J3.1, K3.NC
- new net N$26: D4.A, K3.P$1, T4.E
- net 5V: now also IC1.FB, L1.2; no longer IC1.VO
- net D1: now also R2.2, U1.DATA; no longer D5.A, T1.B
- net D2: now also D5.A, T1.B; no longer D6.A, T2.B
- net D5: now also D6.A, T2.B; no longer R9.1
- net D6: now also D8.A, T3.B; no longer R10.1
- net D7: now also D7.A, T4.B; no longer R8.1
- net GND: now also D10.C, D9.A, IC1.!ON!/OFF, J5.2, J5.3, K1.P$2, K2.P$2, K3.P$2, K4.P$2; no longer D1.C, D10.BLU-C, D10.GRN-C, D10.RED-C, J5.GND, J5.GNDBREAK, K1.COIL2, K2.COIL2, K3.COIL2, K4.COIL2
- net N$1: now also D10.A, K1.P$1; no longer D1.A, K1.COIL1
- net N$10: now also K3.P$4; no longer K3.NO
- net N$11: now also K2.P$5; no longer K2.NC
- net N$12: now also K2.P$3; no longer K2.MAIN
- net N$13: now also K2.P$4; no longer K2.NO
- net N$14: now also K1.P$4; no longer K1.NO
- net N$15: now also K1.P$3; no longer K1.MAIN
- net N$16: now also K1.P$5; no longer K1.NC
- net N$19: now also IC1.VIN, J5.1; no longer IC1.VI, J5.PWR
- net N$2: now also K4.P$5; no longer K4.NC
- net N$23: now also D9.C, IC1.OUT, L1.1; no longer D10.BLU-A, R8.2
- net N$3: now also K2.P$1; no longer K2.COIL1
- net N$4: now also K4.P$3; no longer K4.MAIN
- net N$5: now also K4.P$1; no longer K4.COIL1
- net N$6: now also K4.P$4; no longer K4.NO
- net N$7: now also J3.1, K3.P$5; no longer D4.A, K3.COIL1, T4.E
- net N$9: now also K3.P$3; no longer K3.MAIN
Other:
- note removed: "CONNECTION STATUS"
- moved on the sheet: C1, C2, J2, J4, T2, T3
